Commit message: recursively adding subfolders

File: my_robot/urdf/my_robot.xacro (robot description, xacro)
@@ -170,5 +170,4 @@
       <origin xyz="0 0 0" rpy="0 1.5707 0"/>
       <geometry>
-        <!--box size=".1 .1 .1"/-->
         <mesh filename="package://my_robot/meshes/hokuyo.dae"/>
       </geometry>
@@ -181,4 +180,11 @@
     <axis xyz="0 1 0" rpy="0 0 0"/>
   </joint>
+  <joint name="camera_optical_joint" type="fixed">
+    <origin xyz="0 0 0" rpy="0 0 0"/>
+    <parent link="camera"/>
+    <child link="camera_link_optical"/>
+  </joint>
+  <link name="camera_link_optical">
+  </link>
   <!-- Color scheme-->
   <gazebo reference="chassis">
